File: DJ96_00193E BMS.kicad_sch (KiCad schematic)
At the start: 98 parts, among them CN2 Conn_01x06, P1 Conn_02x02_Top_Bottom, U1 240080

Commit message: U1 update
Parts:
- U1: value 240080 -> RAJ240080
Connections:
- net GND1: now also U1.33
- no-connect marks 19 -> 18
Changed lines of the file:
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@@
   (junction (at 200.66 44.45) (diameter 0) (color 0 0 0 0)
   )
-  (no_connect (at 185.42 86.36))
   (no_connect (at 180.34 86.36))
   (no_connect (at 205.74 86.36))
@@
     (stroke (width 0) (type default) (color 0 0 0 0))
   )
+  (wire (pts (xy 186.69 69.85) (xy 186.69 71.12))
+    (stroke (width 0) (type default) (color 0 0 0 0))
+  )
   (wire (pts (xy 151.13 162.56) (xy 151.13 177.8))
     (stroke (width 0) (type default) (color 0 0 0 0))
@@
     (stroke (width 0) (type default) (color 0 0 0 0))
   )
+  (wire (pts (xy 185.42 86.36) (xy 185.42 69.85))
+    (stroke (width 0) (type default) (color 0 0 0 0))
+  )
   (wire (pts (xy 137.16 127) (xy 139.7 127))
     (stroke (width 0) (type default) (color 0 0 0 0))
@@
     (stroke (width 0) (type default) (color 0 0 0 0))
   )
+  (wire (pts (xy 185.42 69.85) (xy 186.69 69.85))
+    (stroke (width 0) (type default) (color 0 0 0 0))
+  )
   (wire (pts (xy 73.66 30.48) (xy 74.93 30.48))
     (stroke (width 0) (type default) (color 0 0 0 0))
@@
   (symbol (lib_id "DJ96_00193E:240080") (at 190.5 106.68 90) (unit 1)
     (in_bom yes) (on_board yes)
-    (property "Reference" "U1" (id 0) (at 212.09 85.09 90))
-    (property "Value" "240080" (id 1) (at 190.5 104.14 90))
-    (property "Footprint" "" (id 2) (at 185.42 132.08 0)
+    (property "Reference" "U1" (id 0) (at 168.91 85.09 90))
+    (property "Value" "RAJ240080" (id 1) (at 191.77 99.06 90))
+    (property "Footprint" "" (id 2) (at 215.9 111.76 0)
       (effects (font (size 1.27 1.27)) hide)
     )
-    (property "Datasheet" "" (id 3) (at 185.42 132.08 0)
+    (property "Datasheet" "https://www.renesas.com/us/en/document/dst/raj240080-data-sheet?r=501371" (id 3) (at 215.9 111.76 0)
       (effects (font (size 1.27 1.27)) hide)
     )
@@
     (pin "2")
   )
+  (symbol (lib_id "power:GND1") (at 186.69 71.12 0) (unit 1)
+    (in_bom yes) (on_board yes)
+    (property "Reference" "#PWR?" (id 0) (at 186.69 77.47 0)
+      (effects (font (size 1.27 1.27)) hide)
+    )
+    (property "Value" "GND1" (id 1) (at 187.96 74.93 0))
+    (property "Footprint" "" (id 2) (at 186.69 71.12 0)
+      (effects (font (size 1.27 1.27)) hide)
+    )
+    (property "Datasheet" "" (id 3) (at 186.69 71.12 0)
+      (effects (font (size 1.27 1.27)) hide)
+    )
+    (pin "1")
+  )
   (symbol (lib_id "Device:Q_NMOS_GSD") (at 274.32 157.48 270) (unit 1)
     (in_bom yes) (on_board yes)
@@
       (reference "#PWR0119") (unit 1) (value "GND2") (footprint "")
     )
+    (path "/b092d2a9-6b62-4270-9743-3ad356d807ab"
+      (reference "#PWR?") (unit 1) (value "GND1") (footprint "")
+    )
     (path "/5d2db160-74e5-4c2f-8120-6ac0f81d6f09"
       (reference "B1") (unit 1) (value "Thermistor") (footprint "")
@@
     )
     (path "/073a8c45-0262-4cc9-adb7-1d84fbec880b"
-      (reference "U1") (unit 1) (value "240080") (footprint "")
+      (reference "U1") (unit 1) (value "RAJ240080") (footprint "")
     )
     (path "/51a92de3-3300-4b62-bbcf-0078e4df470a"
